Commit message: Comment out camera and grippers

File: motoman_sda10f_support/urdf/sda10f_r2f85_scan.urdf (robot description, URDF)
Before this commit: robot motoman_sda10f, 36 links, 35 joints
Links:
- removed link camera_arm_link
- removed link camera_torso_link
- removed link left_inner_finger
- removed link left_inner_finger_pad
- removed link left_inner_knuckle
- removed link left_outer_finger
- removed link left_outer_knuckle
- removed link motoman_left_ee
- removed link motoman_right_ee
- removed link right_inner_finger
- removed link right_inner_finger_pad
- removed link right_inner_knuckle
- removed link right_outer_finger
- removed link right_outer_knuckle
- removed link robotiq_arg2f_base_link
- removed link robotiq_arg2f_extra_link
Joints:
- removed joint camera_arm_joint
- removed joint camera_torso_joint
- removed joint finger_joint
- removed joint left_inner_finger_joint
- removed joint left_inner_finger_pad_joint
- removed joint left_inner_knuckle_joint
- removed joint left_outer_finger_joint
- removed joint motoman_left_joint_ee
- removed joint motoman_right_joint_ee
- removed joint motoman_right_joint_ee_extra
- removed joint motoman_right_joint_pre_ee
- removed joint right_inner_finger_joint
- removed joint right_inner_finger_pad_joint
- removed joint right_inner_knuckle_joint
- removed joint right_outer_finger_joint
- removed joint right_outer_knuckle_joint
